File: SmartMatrixProtogenShield/KiCAD Project/SmartLED_Shield_Breakout.kicad_pcb (KiCad board)
At the start: 2 copper layers, 45.8 x 38 mm, 23 parts, among them J1 Analog In, P1 Misc. I/O, T1 Teensy 4.0

Commit message: Updated the Shield Breakout to use the Semma QT standard with JST SH headers.
Updated Pinouts to refect current prototracer standards.

Reduced I2c Resistor value to 5.1k to improve high speed performance
Parts:
- added I2C4: JST SM04B, Connector_JST:JST_SH_SM04B-SRSS-TB_1x04-1MP_P1.00mm_Horizontal, F.Cu at (143.5, 86.6)
- I2C1, I2C2, I2C3: value JST S4B-XH-A -> JST SM04B; footprint Connector_JST:JST_XH_S4B-XH-A_1x04_P2.50mm_Horizontal -> Connector_JST:JST_SH_SM04B-SRSS-TB_1x04-1MP_P1.00mm_Horizontal
- R1, R2: value 10k -> 5.1k
- moved I2C3 50.7 mm to (143.5, 77.1)
- moved I2C2 47.6 mm to (143.5, 67.6)
- moved I2C1 44.6 mm to (143.5, 58.1)
- moved B1 42.8 mm to (127.6, 71.0)
- moved C1 42.8 mm to (130.0, 86.5)
- moved C2 42.8 mm to (130.0, 84.0)
- moved C3 42.8 mm to (130.0, 81.5)
- moved C4 42.8 mm to (130.0, 79.0)
- moved J1 42.8 mm to (122.5, 68.5)
- moved BCKPWR1 42.8 mm to (124.9, 80.5)
- moved H1 42.8 mm to (109.4, 57.8)
- moved H2 42.8 mm to (109.4, 86.8)
- moved LED1 42.8 mm to (119.3, 74.4)
- moved LED2 42.8 mm to (119.3, 72.4)
- moved LEDPWR1 42.8 mm to (118.6, 80.5)
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Connections:
- B1 pad 4: /TIO20 -> /TIO23
- I2C1 pad 3: /SCL0 -> /SDA0
- I2C1 pad 4: /SDA0 -> /SCL0
- I2C2 pad 3: /SCL0 -> /SDA0
- I2C2 pad 4: /SDA0 -> /SCL0
- I2C3 pad 3: /SCL0 -> /SDA0
- I2C3 pad 4: /SDA0 -> /SCL0
- P1 pad 16: /TIO23 -> /TIO20
Routing:
- net /TIO23: track 7.62 -> 26.8 mm, vias 0 -> 1
- net /TIO20: track 30.7 -> 13.1 mm
- net /SCL0: track 76.2 -> 86.4 mm, vias 1 -> 2
- net /SDA0: track 93.5 -> 84.6 mm, vias 1 -> 2
- net +3V3: track 122.8 -> 125.6 mm, vias 2 -> 6
- net GND: vias 5 -> 9
Other:
- board size 45.8 x 38 mm -> 45.7 x 38 mm
