File: SmartMatrixProtogenShield/KiCAD Project/SmartLED_Shield_Breakout.kicad_sch (KiCad schematic)
At the start: 23 parts, among them J1 Analog In, P1 Misc. I/O, T1 Teensy 4.0

Commit message: Updated the Shield Breakout to use the Semma QT standard with JST SH headers.
Updated Pinouts to refect current prototracer standards.

Reduced I2c Resistor value to 5.1k to improve high speed performance
Parts:
- added I2C4: JST SM04B, Connector_JST:JST_SH_SM04B-SRSS-TB_1x04-1MP_P1.00mm_Horizontal, symbol Connector_Generic:Conn_01x04
- I2C1, I2C2, I2C3: value JST S4B-XH-A -> JST SM04B; footprint Connector_JST:JST_XH_S4B-XH-A_1x04_P2.50mm_Horizontal -> Connector_JST:JST_SH_SM04B-SRSS-TB_1x04-1MP_P1.00mm_Horizontal
- R1, R2: value 10k -> 5.1k
Connections:
- net +3V3: now also I2C4.2 (Pin_2)
- net GND: now also I2C4.1 (Pin_1)
- net SCL0: now also I2C1.4 (Pin_4), I2C2.4 (Pin_4), I2C3.4 (Pin_4), I2C4.4 (Pin_4); no longer I2C1.3 (Pin_3), I2C2.3 (Pin_3), I2C3.3 (Pin_3)
- net SDA0: now also I2C1.3 (Pin_3), I2C2.3 (Pin_3), I2C3.3 (Pin_3), I2C4.3 (Pin_3); no longer I2C1.4 (Pin_4), I2C2.4 (Pin_4), I2C3.4 (Pin_4)
- net TIO20: now also P1.16 (Pin_16); no longer B1.4 (Pin_4)
- net TIO23: now also B1.4 (Pin_4); no longer P1.16 (Pin_16)
Other:
- company: Coelacanth Electronics, LLC -> Coelacanth Electronics, LLC, Axion Labs, LLC
- moved on the sheet: I2C1, I2C2, I2C3
